Commit message: rviz visualization complete

File: system_bringup/turtle_3d_geometry.urdf (robot description, URDF)
Before this commit: robot turtle1, 1 links, 0 joints
Links:
- removed link turtle_current_pose_frame
- added link turtle_body; visual mesh filename=package://system_bringup/turtle_model.stl scale=0.008 0.008 0.008
